File: SFXboard.brd (EAGLE design)
At the start: 100 x 80 mm, 17 parts, among them J1 AVR_SPI_PRG_62X3_LOCK, J2 POWER_JACKPTH, Q1 16MHz, Q2 BSS138, Q3 BSS138, Q4 BSS138, U1 ATMEGA16U2-AU, X1 USBSMD

Commit message: Layout checkpoint
Parts:
- moved U$2 100.5 mm to (-14.0, 19.1)
- moved J1 35.8 mm to (1.27, 17.8)
- moved C3 24.8 mm to (4.45, 29.2), turned to 270 degrees
- moved X1 24.3 mm to (29.2, 26.0), turned to 180 degrees
- moved Q2 14.0 mm to (15.2, 10.2)
- moved C4 13.9 mm to (17.1, 24.8)
- moved C1 12.5 mm to (17.1, 19.7)
- moved R3 10.3 mm to (22.2, 19.1), turned to 180 degrees
- moved Q1 8.91 mm to (11.4, 29.2), turned to 180 degrees
- moved U1 8.03 mm to (8.89, 21.6)
- moved C2 7.10 mm to (18.4, 29.2), turned to 270 degrees
- moved R1 7.01 mm to (17.1, 22.2), turned to 180 degrees
- moved Q3 6.48 mm to (19.1, 10.2)
- moved R2 2.69 mm to (22.2, 22.2), turned to 180 degrees
- moved Q4 1.80 mm to (22.9, 10.2)
Connections:
- net GRN_PWM: now also Q4.1; no longer Q2.1
- net RED_PWM: now also Q2.1; no longer Q4.1
Routing:
- net N$16: track 0.00 -> 27.7 mm
- net N$2: track 0.00 -> 23.1 mm, vias 0 -> 2
- net N$6: track 0.00 -> 10.7 mm, vias 0 -> 2
- net N$3: track 0.00 -> 10.3 mm
- net N$8: track 0.00 -> 10.1 mm
- net N$9: track 0.00 -> 10.00 mm
- net N$15: track 0.00 -> 9.33 mm
- net N$14: track 0.00 -> 8.30 mm
- net N$10: track 0.00 -> 7.35 mm
- net N$4: track 0.00 -> 6.89 mm
- net N$1: track 0.00 -> 4.97 mm
- net N$5: track 0.00 -> 3.35 mm
- added copper zone on layer 1, net GND
- added copper zone on layer 16, net GND
Other:
- board size 100 x 80 mm -> 34 x 31.7 mm

Commit message: IT IS DONE
Parts:
- moved J1 31.1 mm to (31.8, 11.4), turned to 90 degrees
- moved R3 1.27 mm to (23.5, 19.1)
- moved X1 0.64 mm to (29.2, 25.4)
Routing:
- net N$11: track 0.00 -> 34.2 mm, vias 0 -> 1
- net N$13: track 0.00 -> 31.1 mm, vias 0 -> 1
- net N$12: track 0.00 -> 29.1 mm, vias 0 -> 2
- net N$7: track 0.00 -> 25.0 mm, vias 0 -> 3
- net N$2: track 23.1 -> 38.3 mm
- net GRN_PWM: track 0.00 -> 13.9 mm
- net BLU_PWM: track 0.00 -> 12.8 mm
- net RED_PWM: track 0.00 -> 10.5 mm
- net N$16: track 27.7 -> 26.4 mm
- net N$4: track 6.89 -> 6.25 mm
Other:
- board text added: "Rev 2012-09-16.1"
- board text added: "SFXmachine"
- board text added: "supersat@cs.uw.edu"

Commit message: Smaller OSHW logo
Parts:
- U$2: value OSHW-LOGOL -> OSHW-LOGOS; device SparkFun-Aesthetics:OSHW-LOGO-L -> SparkFun-Aesthetics:OSHW-LOGO-S
Changed lines of the file:
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@@
 <element name="U$1" library="sfxboard" package="TERMBLOCK4P" value="TERMBLOCK4POS" x="22.86" y="3.81"/>
 <element name="J2" library="SparkFun-Connectors" package="POWER_JACK_PTH" value="POWER_JACKPTH" x="5.08" y="0"/>
-<element name="U$2" library="SparkFun-Aesthetics" package="OSHW-LOGO-L" value="OSHW-LOGOL" x="-13.97" y="19.05"/>
+<element name="U$2" library="SparkFun-Aesthetics" package="OSHW-LOGO-S" value="OSHW-LOGOS" x="-13.97" y="19.05"/>
 </elements>
 <signals>
