File: SFXboard.sch (EAGLE design)
At the start: 14 parts, among them J1 AVR_SPI_PRG_62X3_LOCK, Q1 16MHz, Q2 BSS138, Q3 BSS138, Q4 BSS138, U1 ATMEGA16U2-AU, X1 USBSMD

Commit message: Layout checkpoint
Parts:
- added J2: POWER_JACKPTH, SparkFun-Connectors:POWER_JACKPTH
- added U$1: TERMBLOCK4POS, sfxboard:TERMBLOCK4POS
- added U$2: OSHW-LOGOL, SparkFun-Aesthetics:OSHW-LOGOL
Connections:
- new net N$10: Q2.D, U$1.P2
- new net N$14: Q3.D, U$1.P3
- new net N$15: Q4.D, U$1.P4
- new net N$16: J2.PWR, U$1.P1
- net BLU_PWM: now also Q3.G, U1.PC6; no longer Q4.G, U1.PB7
- net GND: now also J2.GND, J2.GNDBREAK
- net GRN_PWM: now also Q4.G; no longer Q3.G
- net RED_PWM: now also U1.PB7; no longer U1.PC6
Changed lines of the file:
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@@
 <part name="J1" library="SparkFun-Connectors" deviceset="AVR_SPI_PRG_6" device="2X3_LOCK"/>
 <part name="GND4" library="supply1" deviceset="GND" device=""/>
+<part name="U$1" library="sfxboard" deviceset="TERMBLOCK4POS" device=""/>
+<part name="J2" library="SparkFun-Connectors" deviceset="POWER_JACK" device="PTH"/>
+<part name="GND5" library="supply1" deviceset="GND" device=""/>
+<part name="U$2" library="SparkFun-Aesthetics" deviceset="OSHW-LOGO" device="L"/>
 </parts>
 <sheets>
@@
 <instance part="J1" gate="G$1" x="50.8" y="25.4"/>
 <instance part="GND4" gate="1" x="63.5" y="12.7"/>
+<instance part="U$1" gate="G$1" x="0" y="73.66"/>
+<instance part="J2" gate="G$1" x="-38.1" y="71.12"/>
+<instance part="GND5" gate="1" x="-33.02" y="68.58"/>
+<instance part="U$2" gate="G$1" x="-55.88" y="-12.7"/>
 </instances>
 <busses>
@@
 <wire x1="60.96" y1="22.86" x2="63.5" y2="22.86" width="0.1524" layer="91"/>
 <wire x1="63.5" y1="22.86" x2="63.5" y2="15.24" width="0.1524" layer="91"/>
+</segment>
+<segment>
+<pinref part="J2" gate="G$1" pin="GNDBREAK"/>
+<wire x1="-35.56" y1="76.2" x2="-33.02" y2="76.2" width="0.1524" layer="91"/>
+<wire x1="-33.02" y1="76.2" x2="-33.02" y2="73.66" width="0.1524" layer="91"/>
+<pinref part="J2" gate="G$1" pin="GND"/>
+<wire x1="-33.02" y1="73.66" x2="-33.02" y2="71.12" width="0.1524" layer="91"/>
+<wire x1="-35.56" y1="73.66" x2="-33.02" y2="73.66" width="0.1524" layer="91"/>
+<pinref part="GND5" gate="1" pin="GND"/>
+<junction x="-33.02" y="73.66"/>
 </segment>
 </net>
@@
 <net name="RED_PWM" class="0">
 <segment>
-<pinref part="U1" gate="G$1" pin="PC6"/>
-<wire x1="20.32" y1="-2.54" x2="35.56" y2="-2.54" width="0.1524" layer="91"/>
-<label x="22.86" y="-2.54" size="1.778" layer="95"/>
+<pinref part="U1" gate="G$1" pin="PB7"/>
+<wire x1="20.32" y1="10.16" x2="35.56" y2="10.16" width="0.1524" layer="91"/>
+<label x="22.86" y="10.16" size="1.778" layer="95"/>
 </segment>
 <segment>
@@
 </net>
 <net name="BLU_PWM" class="0">
-<segment>
-<pinref part="U1" gate="G$1" pin="PB7"/>
-<wire x1="20.32" y1="10.16" x2="35.56" y2="10.16" width="0.1524" layer="91"/>
-<label x="22.86" y="10.16" size="1.778" layer="95"/>
-</segment>
-<segment>
-<pinref part="Q4" gate="G$1" pin="G"/>
-<wire x1="25.4" y1="50.8" x2="25.4" y2="48.26" width="0.1524" layer="91"/>
-<wire x1="25.4" y1="48.26" x2="10.16" y2="48.26" width="0.1524" layer="91"/>
-<label x="10.16" y="48.26" size="1.778" layer="95"/>
-</segment>
-</net>
-<net name="GRN_PWM" class="0">
 <segment>
 <pinref part="Q3" gate="G$1" pin="G"/>
@@
 </segment>
 <segment>
-<pinref part="U1" gate="G$1" pin="PC5"/>
-<wire x1="20.32" y1="0" x2="35.56" y2="0" width="0.1524" layer="91"/>
-<label x="22.86" y="0" size="1.778" layer="95"/>
+<pinref part="U1" gate="G$1" pin="PC6"/>
+<wire x1="20.32" y1="-2.54" x2="35.56" y2="-2.54" width="0.1524" layer="91"/>
+<label x="22.86" y="-2.54" size="1.778" layer="95"/>
 </segment>
 </net>
@@
 </segment>
 </net>
+<net name="N$10" class="0">
+<segment>
+<pinref part="Q2" gate="G$1" pin="D"/>
+<wire x1="-2.54" y1="60.96" x2="-27.94" y2="60.96" width="0.1524" layer="91"/>
+<wire x1="-27.94" y1="60.96" x2="-27.94" y2="55.88" width="0.1524" layer="91"/>
+<pinref part="U$1" gate="G$1" pin="P2"/>
+<wire x1="-2.54" y1="68.58" x2="-2.54" y2="60.96" width="0.1524" layer="91"/>
+</segment>
+</net>
+<net name="N$15" class="0">
+<segment>
+<pinref part="Q4" gate="G$1" pin="D"/>
+<wire x1="7.62" y1="60.96" x2="33.02" y2="60.96" width="0.1524" layer="91"/>
+<wire x1="33.02" y1="60.96" x2="33.02" y2="55.88" width="0.1524" layer="91"/>
+<pinref part="U$1" gate="G$1" pin="P4"/>
+<wire x1="7.62" y1="60.96" x2="7.62" y2="68.58" width="0.1524" layer="91"/>
+</segment>
+</net>
+<net name="N$16" class="0">
+<segment>
+<pinref part="J2" gate="G$1" pin="PWR"/>
+<wire x1="-35.56" y1="78.74" x2="-15.24" y2="78.74" width="0.1524" layer="91"/>
+<wire x1="-15.24" y1="78.74" x2="-15.24" y2="66.04" width="0.1524" layer="91"/>
+<wire x1="-15.24" y1="66.04" x2="-7.62" y2="66.04" width="0.1524" layer="91"/>
+<pinref part="U$1" gate="G$1" pin="P1"/>
+<wire x1="-7.62" y1="66.04" x2="-7.62" y2="68.58" width="0.1524" layer="91"/>
+</segment>
+</net>
+<net name="N$14" class="0">
+<segment>
+<pinref part="U$1" gate="G$1" pin="P3"/>
+<pinref part="Q3" gate="G$1" pin="D"/>
+<wire x1="2.54" y1="68.58" x2="2.54" y2="55.88" width="0.1524" layer="91"/>
+</segment>
+</net>
+<net name="GRN_PWM" class="0">
+<segment>
+<pinref part="Q4" gate="G$1" pin="G"/>
+<wire x1="25.4" y1="50.8" x2="25.4" y2="48.26" width="0.1524" layer="91"/>
+<wire x1="25.4" y1="48.26" x2="10.16" y2="48.26" width="0.1524" layer="91"/>
+<label x="10.16" y="48.26" size="1.778" layer="95"/>
+</segment>
+<segment>
+<pinref part="U1" gate="G$1" pin="PC5"/>
+<wire x1="20.32" y1="0" x2="35.56" y2="0" width="0.1524" layer="91"/>
+<label x="22.86" y="0" size="1.778" layer="95"/>
+</segment>
+</net>

Commit message: Smaller OSHW logo
Parts:
- U$2: value OSHW-LOGOL -> OSHW-LOGOS; device SparkFun-Aesthetics:OSHW-LOGOL -> SparkFun-Aesthetics:OSHW-LOGOS
Changed lines of the file:
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@@
 <part name="J2" library="SparkFun-Connectors" deviceset="POWER_JACK" device="PTH"/>
 <part name="GND5" library="supply1" deviceset="GND" device=""/>
-<part name="U$2" library="SparkFun-Aesthetics" deviceset="OSHW-LOGO" device="L"/>
+<part name="U$2" library="SparkFun-Aesthetics" deviceset="OSHW-LOGO" device="S"/>
 </parts>
 <sheets>
